Commit message: Added Gazebo Model and Gazebo control

File: src/view_robot/urdf/robot.urdf.xacro (robot description, xacro)
@@ -1,6 +1,7 @@
 <?xml version="1.0"?>
-<robot xmlns:xacro="http://www.ros.org/wiki/xacro" name="my_robot">
+<robot xmlns:xacro="http://www.ros.org/wiki/xacro" name="super_robot">
   <xacro:include filename="inertial_macros.xacro"/>
   <xacro:include filename="robot_core.xacro"/>
   <xacro:include filename="robot_sensors.xacro"/>
+  <xacro:include filename="gz_control.xacro"/>
 </robot>

File: src/view_robot/urdf/robot_core.xacro (robot description, xacro)
@@ -34,4 +34,9 @@
     </xacro:inertial_box>
   </link>
+  <gazebo reference="base_plate">
+    <material>
+      Gazebo/White
+    </material>
+  </gazebo>
   <!-- ===== Четыре стойки ===== -->
   <xacro:macro name="rod" params="name x y">
@@ -56,4 +61,9 @@
     </link>
   </xacro:macro>
+  <gazebo reference="rod">
+    <material>
+      Gazebo/Black
+    </material>
+  </gazebo>
   <xacro:rod name="rod_front_left"  x=" 0.09" y=" 0.105"/>
   <xacro:rod name="rod_front_right" x=" 0.09" y="-0.105"/>
@@ -66,4 +76,5 @@
     <origin xyz="0 0.095 0" rpy="0 0 0"/>
     <axis xyz="0 1 0"/>
+    <limit effort="200.0" velocity="20.0"/>
   </joint>
   <link name="left_wheel">
@@ -81,4 +92,9 @@
     </xacro:inertial_cylinder>
   </link>
+  <gazebo reference="left_wheel">
+    <material>
+      Gazebo/Blue
+    </material>
+  </gazebo>
   <joint name="right_wheel_joint" type="continuous">
     <parent link="base_link"/>
@@ -86,4 +102,5 @@
     <origin xyz="0 -0.095 0" rpy="0 0 0"/>
     <axis xyz="0 1 0"/>
+    <limit effort="200.0" velocity="20.0"/>
   </joint>
   <link name="right_wheel">
@@ -101,4 +118,9 @@
     </xacro:inertial_cylinder>
   </link>
+  <gazebo reference="right_wheel">
+    <material>
+      Gazebo/Blue
+    </material>
+  </gazebo>
   <!-- ===== Кастер: было x=-0.09, теперь x=-0.14 ===== -->
   <joint name="caster_wheel_joint" type="fixed">
@@ -121,4 +143,13 @@
     </xacro:inertial_sphere>
   </link>
+  <gazebo reference="caster_wheel">
+    <material>
+      Gazebo/Blue
+    </material>
+    <mu1>0.01</mu1>
+    <mu2>0.01</mu2>
+    <kp>1000000.0</kp>
+    <kd>1.0</kd>
+  </gazebo>
   <!-- ===== Средняя плата электроники ===== -->
   <joint name="electronics_plate_joint" type="fixed">
@@ -141,4 +172,9 @@
     </xacro:inertial_box>
   </link>
+  <gazebo reference="electronic_plate">
+    <material>
+      Gazebo/White
+    </material>
+  </gazebo>
   <!-- ===== Верхняя платформа ===== -->
   <joint name="top_plate_joint" type="fixed">
@@ -161,4 +197,9 @@
     </xacro:inertial_box>
   </link>
+  <gazebo reference="top_plate">
+    <material>
+      Gazebo/White
+    </material>
+  </gazebo>
   <!-- ===== ros2_control ===== -->
   <ros2_control name="my_robot_hardware" type="system">

File: src/view_robot/urdf/robot_sensors.xacro (robot description, xacro)
@@ -45,4 +45,9 @@
     </xacro:inertial_cylinder>
   </link>
+  <gazebo reference="lidar_link">
+    <material>
+      Gazebo/Black
+    </material>
+  </gazebo>
   <!-- ===== Камера ===== -->
   <!--
@@ -79,4 +84,9 @@
     </xacro:inertial_box>
   </link>
+  <gazebo reference="camera_link">
+    <material>
+      Gazebo/Black
+    </material>
+  </gazebo>
   <!--
     camera_optical_frame: стандартный оптический фрейм ROS.
