Commit message: Fixed multiple errors again

File: src/view_robot/urdf/ros2_control.xacro (robot description, xacro)
@@ -20,9 +20,9 @@
             <state_interface name="position"/>
         </joint>
-        <joint name="right wheel_joint">
+        <joint name="right_wheel_joint">
             <command_interface name="velocity">
                 <param name="min">-10</param>
                 <param name="max">10</param>
-            </command interface>
+            </command_interface>
             <state_interface name="velocity"/>
             <state_interface name="position"/>
