Commit message: Fixed URDF and yaml errors

File: src/view_robot/urdf/robot_core.xacro (robot description, xacro)
@@ -2,4 +2,5 @@
 <robot xmlns:xacro="http://www.ros.org/wiki/xacro">
   <xacro:include filename="inertial_macros.xacro"/>
+  <xacro:property name="my_pi" value="${pi if has_property('pi') else 3.14159}" />
   <material name="black">  <color rgba="0 0 0 1"/>       </material>
   <material name="white">  <color rgba="1 1 1 1"/>       </material>
@@ -40,5 +41,5 @@
   </gazebo>
   <!-- ===== Четыре стойки ===== -->
-  <xacro:macro name="rod" params="name x y">
+  <xacro:macro name="rod" params="name x y material_name:=silver gazebo_color:=Gazebo/Black">
     <joint name="${name}_joint" type="fixed">
       <parent link="base_plate"/>
@@ -50,5 +51,5 @@
         <origin xyz="${x} ${y} 0.1" rpy="0 0 0"/>
         <geometry><cylinder length="0.19" radius="0.005"/></geometry>
-        <material name="silver"/>
+        <material name="${material_name}"/>
       </visual>
       <collision>
@@ -61,9 +62,4 @@
     </link>
   </xacro:macro>
-  <gazebo reference="rod">
-    <material>
-      Gazebo/Black
-    </material>
-  </gazebo>
   <xacro:rod name="rod_front_left"  x=" 0.09" y=" 0.105"/>
   <xacro:rod name="rod_front_right" x=" 0.09" y="-0.105"/>
@@ -172,5 +168,5 @@
     </xacro:inertial_box>
   </link>
-  <gazebo reference="electronic_plate">
+  <gazebo reference="electronics_plate">
     <material>
       Gazebo/White
@@ -202,21 +198,3 @@
     </material>
   </gazebo>
-  <!-- ===== ros2_control ===== -->
-  <ros2_control name="my_robot_hardware" type="system">
-    <hardware>
-      <plugin>mock_components/GenericSystem</plugin>
-      <param name="update_rate" type="int">50</param>
-      <param name="calculate_dynamics" type="bool">true</param>
-    </hardware>
-    <joint name="left_wheel_joint">
-      <command_interface name="velocity"/>
-      <state_interface name="position"/>
-      <state_interface name="velocity"/>
-    </joint>
-    <joint name="right_wheel_joint">
-      <command_interface name="velocity"/>
-      <state_interface name="position"/>
-      <state_interface name="velocity"/>
-    </joint>
-  </ros2_control>
 </robot>

File: src/view_robot/urdf/robot_sensors.xacro (robot description, xacro)
@@ -96,12 +96,12 @@
     <visual>
       <origin xyz="0 0 0" rpy="0 0 0"/>
-      <geometry><box size="0.025 0.09 0.025"/></geometry>
+      <geometry><box size="0.025 0.035 0.025"/></geometry>
       <material name="black"/>
     </visual>
     <collision>
       <origin xyz="0 0 0" rpy="0 0 0"/>
-      <geometry><box size="0.025 0.09 0.025"/></geometry>
+      <geometry><box size="0.025 0.035 0.025"/></geometry>
     </collision>
-    <xacro:inertial_box mass="0.1" x="0.025" y="0.09" z="0.025">
+    <xacro:inertial_box mass="0.1" x="0.025" y="0.035" z="0.025">
       <origin xyz="0 0 0" rpy="0 0 0"/>
     </xacro:inertial_box>

Commit message: Added IMU into URDF

File: src/view_robot/urdf/robot_core.xacro (robot description, xacro)
@@ -9,4 +9,10 @@
   <link name="odom"/>
   <link name="base_link"/>
+  <joint name="base_footprint_joint" type="fixed">
+    <parent link="base_link"/>
+    <child link="base_footprint"/>
+    <origin xyz="0 0 0" rpy="0 0 0"/>
+  </joint>
+  <link name="base_footprint"></link>
   <joint name="base_link_joint" type="fixed">
     <parent link="odom"/>

File: src/view_robot/urdf/robot_sensors.xacro (robot description, xacro)
@@ -125,3 +125,22 @@
   </joint>
   <link name="camera_optical_frame"/>
+  <joint name="imu_link" type="fixed">
+    <parent link="base_link"/>
+    <child link="imu_link"/>
+    <origin xyz="-0.016 0.032 -0.007" rpy="0 0 -3.14159"/>
+  </joint>
+  <link name="imu_link">
+    <visual>
+      <origin xyz="-0.016 0.032 -0.007" rpy="0 0 -3.14159"/>
+      <geometry><box size="0.015 0.02 0.003"/></geometry>
+      <material name="black"/>
+    </visual>
+    <collision>
+      <origin xyz="-0.016 0.032 -0.007" rpy="0 0 -3.14159"/>
+      <geometry><box size="0.015 0.02 0.003"/></geometry>
+    </collision>
+    <xacro:inertial_box mass="0.002" x="0.015" y="0.02" z="0.003">
+       <origin xyz="-0.016 0.032 -0.007" rpy="0 0 -3.14159"/>
+    </xacro:inertial_box>
+  </link>
 </robot>
