Commit message: Добавил ROS2 Control

File: src/view_robot/urdf/robot_sensors.xacro (robot description, xacro)
@@ -7,4 +7,5 @@
     <child link="lidar_base"/>
     <origin xyz="0 0 0.005" rpy="0 0 0"/>
+    <preserveFixedJoint>true</preserveFixedJoint>
   </joint>
   <link name="lidar_base">
@@ -29,5 +30,9 @@
     <child link="lidar_link"/>
     <origin xyz="0 0 0.02988" rpy="0 0 0"/>
+    <preserveFixedJoint>true</preserveFixedJoint>
   </joint>
+  <gazebo reference="lidar_joint">
+    <preserveFixedJoint>true</preserveFixedJoint>
+  </gazebo>
   <link name="lidar_link">
     <visual>
@@ -46,7 +51,25 @@
   </link>
   <gazebo reference="lidar_link">
-    <material>
-      Gazebo/Black
-    </material>
+    <sensor name="gpu_lidar" type="gpu_lidar">
+      <topic>/scan_gz</topic>
+      <update_rate>10</update_rate>
+      <lidar>
+        <scan>
+          <horizontal>
+            <samples>360</samples>
+            <resolution>1</resolution>
+            <min_angle>-3.14159</min_angle>
+            <max_angle>3.14159</max_angle>
+          </horizontal>
+        </scan>
+        <range>
+          <min>0.05</min>
+          <max>12.0</max>
+          <resolution>0.01</resolution>
+        </range>
+      </lidar>
+      <always_on>true</always_on>
+      <visualize>true</visualize>
+    </sensor>
   </gazebo>
   <!-- ===== Камера ===== -->

Commit message: Added IMU into EKF and updated DiffDrive plpugin for Ros2 Control Package

File: src/view_robot/urdf/robot_sensors.xacro (robot description, xacro)
@@ -132,14 +132,14 @@
   <link name="imu_link">
     <visual>
-      <origin xyz="-0.016 0.032 -0.007" rpy="0 0 -3.14159"/>
+      <origin xyz="0 0 0" rpy="0 0 0"/>
       <geometry><box size="0.015 0.02 0.003"/></geometry>
       <material name="black"/>
     </visual>
     <collision>
-      <origin xyz="-0.016 0.032 -0.007" rpy="0 0 -3.14159"/>
+      <origin xyz="0 0 0" rpy="0 0 0"/>
       <geometry><box size="0.015 0.02 0.003"/></geometry>
     </collision>
     <xacro:inertial_box mass="0.002" x="0.015" y="0.02" z="0.003">
-       <origin xyz="-0.016 0.032 -0.007" rpy="0 0 -3.14159"/>
+       <origin xyz="0 0 0" rpy="0 0 0"/>
     </xacro:inertial_box>
   </link>
